File: led_array_driver/led_array_driver.kicad_sch (KiCad schematic)
At the start: 0 parts

Commit message: 1
Parts:
- added IC1: MP24894GJ-P, SOP95P280X100-6N, symbol MP24894:MP24894GJ-P
Changed lines of the file:
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@@
     (company "PED - AHL")
+  )
+  (symbol (lib_id "power:GND") (at 19.05 25.4 0) (unit 1)
+    (in_bom yes) (on_board yes) (dnp no) (fields_autoplaced)
+    (property "Reference" "#PWR02" (at 19.05 31.75 0)
+      (effects (font (size 1.27 1.27)) hide)
+    )
+    (property "Value" "GND" (at 19.05 30.48 0)
+      (effects (font (size 1.27 1.27)))
+    )
+    (property "Footprint" "" (at 19.05 25.4 0)
+      (effects (font (size 1.27 1.27)) hide)
+    )
+    (property "Datasheet" "" (at 19.05 25.4 0)
+      (effects (font (size 1.27 1.27)) hide)
+    )
+    (pin "1")
+    (instances
+      (project "led_array_driver"
+        (path "/be3a2376-e359-421d-aadd-cbde73488a33"
+          (reference "#PWR02") (unit 1)
+        )
+      )
+    )
+  )
+  (symbol (lib_id "power:+12V") (at 27.94 27.94 0) (unit 1)
+    (in_bom yes) (on_board yes) (dnp no) (fields_autoplaced)
+    (property "Reference" "#PWR01" (at 27.94 31.75 0)
+      (effects (font (size 1.27 1.27)) hide)
+    )
+    (property "Value" "+12V" (at 27.94 24.13 0)
+      (effects (font (size 1.27 1.27)))
+    )
+    (property "Footprint" "" (at 27.94 27.94 0)
+      (effects (font (size 1.27 1.27)) hide)
+    )
+    (property "Datasheet" "" (at 27.94 27.94 0)
+      (effects (font (size 1.27 1.27)) hide)
+    )
+    (pin "1")
+    (instances
+      (project "led_array_driver"
+        (path "/be3a2376-e359-421d-aadd-cbde73488a33"
+          (reference "#PWR01") (unit 1)
+        )
+      )
+    )
+  )
+  (symbol (lib_id "MP24894:MP24894GJ-P") (at 43.18 39.37 0) (unit 1)
+    (in_bom yes) (on_board yes) (dnp no) (fields_autoplaced)
+    (property "Reference" "IC1" (at 58.42 33.02 0)
+      (effects (font (size 1.27 1.27)))
+    )
+    (property "Value" "MP24894GJ-P" (at 58.42 35.56 0)
+      (effects (font (size 1.27 1.27)))
+    )
+    (property "Footprint" "SOP95P280X100-6N" (at 69.85 36.83 0)
+      (effects (font (size 1.27 1.27)) (justify left) hide)
+    )
+    (property "Datasheet" "https://componentsearchengine.com/Datasheets/1/MP24894GJ-P.pdf" (at 69.85 39.37 0)
+      (effects (font (size 1.27 1.27)) (justify left) hide)
+    )
+    (property "Description" "Monolithic Power Systems (MPS) MP24894GJ-P LED Driver IC, 6  60 V 6-Pin TSOT" (at 69.85 41.91 0)
+      (effects (font (size 1.27 1.27)) (justify left) hide)
+    )
+    (property "Height" "1" (at 69.85 44.45 0)
+      (effects (font (size 1.27 1.27)) (justify left) hide)
+    )
+    (property "Manufacturer_Name" "Monolithic Power Systems (MPS)" (at 69.85 46.99 0)
+      (effects (font (size 1.27 1.27)) (justify left) hide)
+    )
+    (property "Manufacturer_Part_Number" "MP24894GJ-P" (at 69.85 49.53 0)
+      (effects (font (size 1.27 1.27)) (justify left) hide)
+    )
+    (property "Mouser Part Number" "946-MP24894GJP" (at 69.85 52.07 0)
+      (effects (font (size 1.27 1.27)) (justify left) hide)
+    )
+    (property "Mouser Price/Stock" "https://www.mouser.co.uk/ProductDetail/Monolithic-Power-Systems-MPS/MP24894GJ-P?qs=Iq7RKQRjpgqwFz9droqB6g%3D%3D" (at 69.85 54.61 0)
+      (effects (font (size 1.27 1.27)) (justify left) hide)
+    )
+    (property "Arrow Part Number" "" (at 69.85 57.15 0)
+      (effects (font (size 1.27 1.27)) (justify left) hide)
+    )
+    (property "Arrow Price/Stock" "" (at 69.85 59.69 0)
+      (effects (font (size 1.27 1.27)) (justify left) hide)
+    )
+    (pin "1")
+    (pin "2")
+    (pin "3")
+    (pin "4")
+    (pin "5")
+    (pin "6")
+    (instances
+      (project "led_array_driver"
+        (path "/be3a2376-e359-421d-aadd-cbde73488a33"
+          (reference "IC1") (unit 1)
+        )
+      )
+    )
   )
   (sheet_instances
